File: H12/EtherCAT _Shield/EtherCAT_Shield.kicad_sch (KiCad schematic)
At the start: 33 parts, among them J1 Conn_02x15_Odd_Even, J2 Conn_02x10_Odd_Even, J4 Conn_02x17_Odd_Even, J5 Conn_02x08_Odd_Even, SW1 RESET, U1 LAN9252I/PT, U2 24AA64T-E/OT, Y1 Crystal

Commit message: SQI_SCK Net Labeling correction
Connections:
- net SQI_CLK is gone; now on net SQI_SCK: J4.15 (Pin_15)
Other:
- moved on the sheet: C1, C2
